File: Hardware/Battery Tester/Battery Tester.kicad_sch (KiCad schematic)
At the start: 16 parts, among them J1 USB4105-GF-A, J2 Conn_01x02_Socket, SW1 SW_SPST, U1 MCP73831-5-OT, U2 LP5907MFX-3.3_NOPB

Commit message: hardware updates
Parts:
- R1: value 2k -> 2.5k
Changed lines of the file:
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@@
+		)
+	)
+	(bus_entry
+		(at 102.87 21.59)
+		(size 2.54 2.54)
+		(stroke
+			(width 0)
+			(type default)
+		)
+	)
+	(bus_entry
+		(at 102.87 20.32)
+		(size 2.54 2.54)
+		(stroke
+			(width 0)
+			(type default)
 		)
 	)
@@
 			)
 		)
-		(property "Value" "2k"
+		(property "Value" "2.5k"
 			(at 114.3 48.2599 0)
 			(effects
